File: SD2IECplug.kicad_pcb (KiCad board)
At the start: 2 copper layers, 50 x 88 mm, 61 parts, among them J1 ISP, J2 LED, J3 SD_Card, J4 IEC, J5 C64-CassettePort, J6 C64-CassettePort, J7 USB_B, J8 I2C, J9 SW, Q1 IRLML2803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

Commit message: First steps.
Parts:
- removed J9: SW, Pin_Headers:Pin_Header_Straight_1x06_Pitch2.54mm
- removed R16, R17, R21: 10k, Capacitors_SMD:C_0805_HandSoldering
- removed R18, R19: 22k, Capacitors_SMD:C_0805_HandSoldering
- removed R20: 470, Capacitors_SMD:C_0805_HandSoldering
- removed REF** (x9): VIA-0.6mm, hackup:VIA-0.6mm
- removed REF** (x5): 1pin, Connectors:1pin
- removed U3: PC817, hackup:SOP-4
- D3: value 1N4148 -> 1N5817; footprint Diodes_SMD:D_MicroMELF_Hadsoldering -> Diodes_THT:D_DO-41_SOD81_P7.62mm_Horizontal
- J2: value LED -> X6; footprint Pin_Headers:Pin_Header_Straight_1x04_Pitch2.54mm -> Pin_Headers:Pin_Header_Straight_1x05_Pitch2.54mm
- J7: value USB_B -> Power; footprint Connectors:USB_Mini-B -> Pin_Headers:Pin_Header_Straight_1x02_Pitch2.54mm; moved to F.Cu
- J8: value I2C -> X3; footprint Pin_Headers:Pin_Header_Straight_1x04_Pitch2.54mm -> Pin_Headers:Pin_Header_Straight_1x10_Pitch2.54mm
- moved J7 77.0 mm to (135.7, 76.4)
- moved J8 49.9 mm to (128.4, 76.4), turned to 0 degrees
- moved J4 37.9 mm to (31.3, 115.2)
- moved J2 26.1 mm to (132.1, 76.4)
Connections:
- D1 pad 2: Net-(D1-Pad2) -> /LED2
- D2 pad 2: Net-(D2-Pad2) -> /LED1
- J2 pad 1: Net-(D1-Pad2) -> Net-(J2-Pad1)
- J2 pad 2: Net-(D2-Pad2) -> Net-(J2-Pad2)
- J2 pad 3: Cas-GND -> Net-(J2-Pad3)
- J2 pad 4: (no net) -> Net-(J2-Pad4)
- J7 pad 1: Net-(C4-Pad1) -> Cas-GND
- J7 pad 2: Net-(J7-Pad2) -> Cas-5V
- J8 pad 1: SDA -> /DISKSWITCH
- J8 pad 2: SCL -> Cas-GND
- J8 pad 3: Cas-GND -> /RESERVE
- J8 pad 4: +3V3 -> /LED1
- R1 pad 1: Net-(D1-Pad2) -> /LED2
- R1 pad 2: SCL -> Net-(R1-Pad2)
- R5 pad 1: Net-(D2-Pad2) -> /LED1
- R5 pad 2: SDA -> Net-(R5-Pad2)
- U1 pad 14: Net-(R17-Pad1) -> /IEC_10-11
- U1 pad 16: Net-(U1-Pad16) -> /IEC_8-9
- U1 pad 19: SCL -> Net-(R1-Pad2)
- U1 pad 20: SDA -> Net-(R5-Pad2)
- U1 pad 21: Net-(U1-Pad21) -> /RESERVE
- U1 pad 22: Net-(J9-Pad1) -> /DISKSWITCH
- U1 pad 23: Net-(J9-Pad2) -> Net-(J2-Pad4)
- U1 pad 24: Net-(J9-Pad3) -> Net-(J2-Pad3)
- U1 pad 25: Net-(J9-Pad4) -> Net-(J2-Pad2)
- U1 pad 26: Net-(J9-Pad5) -> Net-(J2-Pad1)
Routing:
- net Cas-5V: track 134.6 -> 0.00 mm, vias 2 -> 0
- net Cas-Write: track 130.6 -> 0.00 mm, vias 4 -> 0
- net +3V3: track 128.3 -> 0.00 mm, vias 8 -> 0
- net Cas-Read: track 127.7 -> 0.00 mm, vias 4 -> 0
- net Cas-Motor: track 126.7 -> 0.00 mm, vias 5 -> 0
- net Cas-Sense: track 117.8 -> 0.00 mm, vias 3 -> 0
- net Net-(U1-Pad13): track 48.4 -> 0.00 mm, vias 3 -> 0
- net Net-(Q2-Pad1): track 44.1 -> 0.00 mm, vias 3 -> 0
- net Net-(R13-Pad2): track 42.7 -> 0.00 mm, vias 3 -> 0
- net Net-(R10-Pad2): track 41.8 -> 0.00 mm, vias 3 -> 0
- net Net-(R3-Pad2): track 40.6 -> 0.00 mm, vias 3 -> 0
- net Net-(Q4-Pad1): track 37.2 -> 0.00 mm, vias 3 -> 0
- net SCK: track 37.1 -> 0.00 mm, vias 2 -> 0
- net SCL: track 36.1 -> 0.00 mm, vias 2 -> 0
- net SDA: track 36.0 -> 0.00 mm, vias 2 -> 0
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
Commit message: First routing.
Parts:
- removed J3: SD_Card, SD-Connectors:SD-Connector-Short
- added XS1: SD Connector, lib:Conn_uSDcard, F.Cu at (103.2, 116.8)
- D3: moved to F.Cu
- moved J7 91.4 mm to (59.5, 126.9)
- moved J2 56.8 mm to (105.6, 126.7)
- moved J1 55.1 mm to (101.9, 134.3)
- moved J8 54.3 mm to (82.6, 105.6), turned to 90 degrees
- moved Y1 54.2 mm to (67.0, 129.5)
- moved C1 54.2 mm to (73.0, 125.5)
- moved C2 54.2 mm to (65.7, 125.5)
- moved C4 50.7 mm to (98.3, 124.3)
- moved C5 50.7 mm to (98.3, 110.8)
- moved C6 50.7 mm to (99.8, 113.8)
- moved U2 50.7 mm to (97.8, 118.8)
- moved D3 49.2 mm to (101.7, 127.2), turned to 180 degrees
- moved C3 46.2 mm to (105.7, 113.7)
- moved R15 46.2 mm to (105.7, 120.6)
- moved D1 45.5 mm to (87.8, 112.9)
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Connections:
- C3 pad 2: Cas-GND -> Net-(C3-Pad2)
- J4 pad 6: Net-(J4-Pad6) -> (no net)
- U1 pad 10: Net-(U1-Pad10) -> (no net)
- U1 pad 12: Net-(U1-Pad12) -> (no net)
- U1 pad 13: Net-(U1-Pad13) -> (no net)
- U1 pad 15: Net-(J3-Pad11) -> Cas-GND
- U1 pad 29: Net-(U1-Pad29) -> (no net)
- U1 pad 40: Net-(U1-Pad40) -> (no net)
- U1 pad 41: Net-(U1-Pad41) -> (no net)
- U1 pad 42: Net-(U1-Pad42) -> (no net)
- U1 pad 43: Net-(U1-Pad43) -> (no net)
- U1 pad 9: Net-(U1-Pad9) -> (no net)
Routing:
- net Cas-5V: track 0.00 -> 99.1 mm, vias 0 -> 4
- net Cas-Motor: track 0.00 -> 86.1 mm, vias 0 -> 2
- net Cas-Read: track 0.00 -> 80.4 mm, vias 0 -> 2
- net +3V3: track 0.00 -> 78.6 mm, vias 0 -> 5
- net Cas-Write: track 0.00 -> 74.2 mm, vias 0 -> 2
- net Cas-Sense: track 0.00 -> 66.4 mm, vias 0 -> 2
- net Cas-GND: track 0.00 -> 54.6 mm, vias 0 -> 17
- net /IEC_10-11: track 0.00 -> 39.0 mm, vias 0 -> 2
- net MOSI: track 0.00 -> 37.3 mm, vias 0 -> 1
- net /IEC_8-9: track 0.00 -> 34.7 mm, vias 0 -> 2
- net SCK: track 0.00 -> 30.7 mm, vias 0 -> 2
- net /RESERVE: track 0.00 -> 29.9 mm
- net Net-(J2-Pad4): track 0.00 -> 29.3 mm
- net Net-(R10-Pad2): track 0.00 -> 29.2 mm, vias 0 -> 3
- net MISO: track 0.00 -> 29.1 mm, vias 0 -> 3
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Other:
- board size 50 x 88 mm -> 50 x 49 mm
- net class Default: clearance 0.2 -> 0.18; trace_width 0.25 -> 0.2; via_dia 0.6 -> 0.45; via_drill 0.4 -> 0.3
- net class PassThru removed
- net class Power added: clearance 0.2, trace_width 0.4, via_dia 0.8, via_drill 0.4
- rule trace_clearance: 0.2 -> 0.18
- board text added: "SD2IEC Pluggable - V2.0"
- board text removed: "SD2IEC Pluggable - V0.9"
