File: SD2IECplug.sch (KiCad schematic (older format))
At the start: 39 parts, among them J1 ISP, J2 X6, J4 IEC, J5 C64-CassettePort, J6 C64-CassettePort, J7 Power, J8 X3, Q1 IRLML2803, Q2 IRLML2803, Q3 IRLML2803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

Commit message: Ziptie holes and silk screen cleanup.
Parts:
- added MH1, MH2: ZipTie, DIN-Connectors:ZipTie_2.7mm, symbol Mechanical:MountingHole
- J4: footprint DIN-Connectors:DIN-6 -> DIN-Connectors:DIN-6-Variable
Changed lines of the file:
@@
 F 0 "J4" H 10325 1425 50  0000 C CNN
 F 1 "IEC" H 10350 950 50  0000 L CNN
-F 2 "DIN-Connectors:DIN-6" H 10200 1200 50  0001 C CNN
+F 2 "DIN-Connectors:DIN-6-Variable" H 10200 1200 50  0001 C CNN
 F 3 "" H 10200 1200 50  0001 C CNN
 	1    10200 1200
@@
 Text Label 3400 6000 0    39   ~ 0
 WRITE_PROTECT
+$Comp
+L Mechanical:MountingHole MH1
+U 1 1 5B9A6E0D
+P 10500 6050
+F 0 "MH1" H 10600 6096 50  0000 L CNN
+F 1 "ZipTie" H 10600 6005 50  0000 L CNN
+F 2 "DIN-Connectors:ZipTie_2.7mm" H 10500 6050 50  0001 C CNN
+F 3 "~" H 10500 6050 50  0001 C CNN
+	1    10500 6050
+	1    0    0    -1
+$EndComp
+$Comp
+L Mechanical:MountingHole MH2
+U 1 1 5B9A6EE3
+P 10500 6200
+F 0 "MH2" H 10600 6246 50  0000 L CNN
+F 1 "ZipTie" H 10600 6155 50  0000 L CNN
+F 2 "DIN-Connectors:ZipTie_2.7mm" H 10500 6200 50  0001 C CNN
+F 3 "~" H 10500 6200 50  0001 C CNN
+	1    10500 6200
+	1    0    0    -1
+$EndComp
 $EndSCHEMATC

Commit message: Added missing resistor and yet another breakout header.
Parts:
- added J3: Aux, Pin_Headers:Pin_Header_Straight_1x03_Pitch2.54mm, symbol conn:Conn_01x03
- added R16: nB, Resistors_SMD:R_0805_HandSoldering, symbol device:R
Connections:
- wire segments 154 -> 165
Changed lines of the file:
@@
 Connection ~ 4100 1450
-Wire Wire Line
-	4500 2700 3400 2700
 Wire Wire Line
 	3800 3100 3400 3100
@@
 	1    0    0    -1
 $EndComp
+$Comp
+L conn:Conn_01x03 J3
+U 1 1 5B9BC1D8
+P 4450 3700
+F 0 "J3" H 4530 3742 50  0000 L CNN
+F 1 "Aux" H 4530 3651 50  0000 L CNN
+F 2 "Pin_Headers:Pin_Header_Straight_1x03_Pitch2.54mm" H 4450 3700 50  0001 C CNN
+F 3 "~" H 4450 3700 50  0001 C CNN
+	1    4450 3700
+	1    0    0    -1
+$EndComp
+$Comp
+L device:R R16
+U 1 1 5B9BC306
+P 3750 3500
+F 0 "R16" V 3700 3300 50  0000 C CNN
+F 1 "nB" V 3750 3500 50  0000 C CNN
+F 2 "Resistors_SMD:R_0805_HandSoldering" V 3680 3500 50  0001 C CNN
+F 3 "~" H 3750 3500 50  0001 C CNN
+	1    3750 3500
+	0    1    1    0
+$EndComp
+Wire Wire Line
+	3400 3800 3550 3800
+Wire Wire Line
+	3550 3800 3550 3500
+Wire Wire Line
+	3550 3500 3600 3500
+Wire Wire Line
+	3400 3600 4250 3600
+Wire Wire Line
+	3400 3700 4250 3700
+Wire Wire Line
+	3400 3900 3950 3900
+Wire Wire Line
+	3950 3900 3950 3800
+Wire Wire Line
+	3950 3800 4250 3800
+Wire Wire Line
+	3400 2700 4050 2700
+Wire Wire Line
+	4050 3500 4050 2700
+Wire Wire Line
+	3900 3500 4050 3500
+Connection ~ 4050 2700
+Wire Wire Line
+	4050 2700 4500 2700
 $EndSCHEMATC

Commit message: Added mounting hole.
Parts:
- added MH3: MountingHole, Mounting_Holes:MountingHole_2.7mm_M2.5, symbol Mechanical:MountingHole
Changed lines of the file:
@@
 Wire Wire Line
 	4050 2700 4500 2700
+$Comp
+L Mechanical:MountingHole MH3
+U 1 1 5B9F7C3B
+P 9750 6200
+F 0 "MH3" H 9850 6246 50  0000 L CNN
+F 1 "MountingHole" H 9850 6155 50  0000 L CNN
+F 2 "Mounting_Holes:MountingHole_2.7mm_M2.5" H 9750 6200 50  0001 C CNN
+F 3 "~" H 9750 6200 50  0001 C CNN
+	1    9750 6200
+	1    0    0    -1
+$EndComp
 $EndSCHEMATC

Commit message: Aligned external power connector.
Parts:
- added MH4: MountingHole, Mounting_Holes:MountingHole_2.7mm_M2.5, symbol Mechanical:MountingHole
Changed lines of the file:
@@
 L Mechanical:MountingHole MH3
 U 1 1 5B9F7C3B
+P 9750 6050
+F 0 "MH3" H 9850 6096 50  0000 L CNN
+F 1 "MountingHole" H 9850 6005 50  0000 L CNN
+F 2 "Mounting_Holes:MountingHole_2.7mm_M2.5" H 9750 6050 50  0001 C CNN
+F 3 "~" H 9750 6050 50  0001 C CNN
+	1    9750 6050
+	1    0    0    -1
+$EndComp
+$Comp
+L Mechanical:MountingHole MH4
+U 1 1 5BA07AD8
 P 9750 6200
-F 0 "MH3" H 9850 6246 50  0000 L CNN
+F 0 "MH4" H 9850 6246 50  0000 L CNN
 F 1 "MountingHole" H 9850 6155 50  0000 L CNN
 F 2 "Mounting_Holes:MountingHole_2.7mm_M2.5" H 9750 6200 50  0001 C CNN

Commit message: Added decoupling cap.
Parts:
- added C7: 100n, Capacitors_SMD:C_0805_HandSoldering, symbol device:C
Connections:
- wire segments 165 -> 166
Changed lines of the file:
@@
+	1    0    0    -1
+$EndComp
+$Comp
+L device:C C7
+U 1 1 5BA17687
+P 1250 6300
+F 0 "C7" H 1365 6346 50  0000 L CNN
+F 1 "100n" H 1365 6255 50  0000 L CNN
+F 2 "Capacitors_SMD:C_0805_HandSoldering" H 1288 6150 50  0001 C CNN
+F 3 "~" H 1250 6300 50  0001 C CNN
+	1    1250 6300
+	1    0    0    -1
+$EndComp
+Wire Wire Line
+	2100 6450 1250 6450
+Connection ~ 2100 6450
+$Comp
+L power:+3V3 #PWR0104
+U 1 1 5BA1F62D
+P 1250 6150
+F 0 "#PWR0104" H 1250 6000 50  0001 C CNN
+F 1 "+3V3" H 1250 6290 50  0000 C CNN
+F 2 "" H 1250 6150 50  0001 C CNN
+F 3 "" H 1250 6150 50  0001 C CNN
+	1    1250 6150
 	1    0    0    -1
 $EndComp

Commit message: Added push buttons.
Parts:
- added SW1, SW2: SW_Push, Buttons_Switches_SMD:SW_SPST_FSMSM, symbol Switch:SW_Push
Connections:
- wire segments 166 -> 170
Changed lines of the file:
@@
 	1    0    0    -1
 $EndComp
+$Comp
+L Switch:SW_Push SW1
+U 1 1 5B99DC09
+P 8500 1100
+F 0 "SW1" H 8500 1385 50  0000 C CNN
+F 1 "SW_Push" H 8500 1294 50  0000 C CNN
+F 2 "Buttons_Switches_SMD:SW_SPST_FSMSM" H 8500 1300 50  0001 C CNN
+F 3 "" H 8500 1300 50  0001 C CNN
+	1    8500 1100
+	1    0    0    -1
+$EndComp
+$Comp
+L Switch:SW_Push SW2
+U 1 1 5B99DF83
+P 8500 1500
+F 0 "SW2" H 8500 1785 50  0000 C CNN
+F 1 "SW_Push" H 8500 1694 50  0000 C CNN
+F 2 "Buttons_Switches_SMD:SW_SPST_FSMSM" H 8500 1700 50  0001 C CNN
+F 3 "" H 8500 1700 50  0001 C CNN
+	1    8500 1500
+	1    0    0    -1
+$EndComp
+Text Label 8300 1100 2    39   ~ 0
+DISKSWITCH
+Text Label 8300 1500 2    39   ~ 0
+RESERVE
+$Comp
+L power:GND #PWR0105
+U 1 1 5B9A5F75
+P 8750 1550
+F 0 "#PWR0105" H 8750 1300 50  0001 C CNN
+F 1 "GND" H 8750 1400 50  0000 C CNN
+F 2 "" H 8750 1550 50  0001 C CNN
+F 3 "" H 8750 1550 50  0001 C CNN
+	1    8750 1550
+	1    0    0    -1
+$EndComp
+Wire Wire Line
+	8700 1100 8750 1100
+Wire Wire Line
+	8750 1100 8750 1500
+Wire Wire Line
+	8700 1500 8750 1500
+Connection ~ 8750 1500
+Wire Wire Line
+	8750 1500 8750 1550
 $EndSCHEMATC

Commit message: Improved ziptie holes.
Parts:
- MH1, MH2: footprint DIN-Connectors:ZipTie_2.7mm -> DIN-Connectors:ZipTie_3.0mm
Changed lines of the file:
@@
 F 0 "MH1" H 10600 6096 50  0000 L CNN
 F 1 "ZipTie" H 10600 6005 50  0000 L CNN
-F 2 "DIN-Connectors:ZipTie_2.7mm" H 10500 6050 50  0001 C CNN
+F 2 "DIN-Connectors:ZipTie_3.0mm" H 10500 6050 50  0001 C CNN
 F 3 "~" H 10500 6050 50  0001 C CNN
 	1    10500 6050
@@
 F 0 "MH2" H 10600 6246 50  0000 L CNN
 F 1 "ZipTie" H 10600 6155 50  0000 L CNN
-F 2 "DIN-Connectors:ZipTie_2.7mm" H 10500 6200 50  0001 C CNN
+F 2 "DIN-Connectors:ZipTie_3.0mm" H 10500 6200 50  0001 C CNN
 F 3 "~" H 10500 6200 50  0001 C CNN
 	1    10500 6200

Commit message: IRLML2803 -> BSS138
Parts:
- Q1, Q2, Q3, Q4: value IRLML2803 -> BSS138
Changed lines of the file:
@@
 P 6700 1800
 F 0 "Q4" H 6900 1875 50  0000 L CNN
-F 1 "IRLML2803" H 6350 1950 50  0000 L CNN
+F 1 "BSS138" H 6450 1950 50  0000 L CNN
 F 2 "TO_SOT_Packages_SMD:SOT-23_Handsoldering" H 6900 1725 50  0001 L CIN
 F 3 "" H 6700 1800 50  0001 L CNN
@@
 P 5800 1800
 F 0 "Q3" H 6000 1875 50  0000 L CNN
-F 1 "IRLML2803" H 5450 1950 50  0000 L CNN
+F 1 "BSS138" H 5550 1950 50  0000 L CNN
 F 2 "TO_SOT_Packages_SMD:SOT-23_Handsoldering" H 6000 1725 50  0001 L CIN
 F 3 "" H 5800 1800 50  0001 L CNN
@@
 P 4900 1800
 F 0 "Q2" H 5100 1875 50  0000 L CNN
-F 1 "IRLML2803" H 4550 1950 50  0000 L CNN
+F 1 "BSS138" H 4650 1950 50  0000 L CNN
 F 2 "TO_SOT_Packages_SMD:SOT-23_Handsoldering" H 5100 1725 50  0001 L CIN
 F 3 "" H 4900 1800 50  0001 L CNN
@@
 P 4000 1800
 F 0 "Q1" H 4200 1875 50  0000 L CNN
-F 1 "IRLML2803" H 3650 1950 50  0000 L CNN
+F 1 "BSS138" H 3750 1950 50  0000 L CNN
 F 2 "TO_SOT_Packages_SMD:SOT-23_Handsoldering" H 4200 1725 50  0001 L CIN
 F 3 "" H 4000 1800 50  0001 L CNN
