File: SD2IECplug.sch (KiCad schematic (older format))
At the start: 48 parts, among them J1 ISP, J2 X6, J3 Aux, J4 IEC, J5 C64-CassettePort, J6 C64-CassettePort, J7 Power, J8 X3, Q1 BSS138, Q2 BSS138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

Commit message: Corrected LED numbering.
Parts:
- U2: value LM1117-3.3 -> AMS1117-3.3
- renumbered D2 to D1, D1 to D2
Changed lines of the file:
@@
 Sheet 1 1
 Title "SD2IEC Pluggable"
-Date "2018-09-10"
-Rev "2.0"
+Date "2018-10-14"
+Rev "2.1"
 Comp "www.hackup.net"
 Comment1 ""
@@
 P 9850 2400
 F 0 "U2" H 9700 2525 50  0000 C CNN
-F 1 "LM1117-3.3" H 9850 2525 50  0000 L CNN
+F 1 "AMS1117-3.3" H 9850 2525 50  0000 L CNN
 F 2 "TO_SOT_Packages_SMD:SOT-223-3_TabPin2" H 9850 2400 50  0001 C CNN
 F 3 "" H 9850 2400 50  0001 C CNN
@@
 $EndComp
 $Comp
-L device:LED D1
+L device:LED D2
 U 1 1 5A0E5986
 P 4200 4500
-F 0 "D1" H 4200 4600 50  0000 C CNN
+F 0 "D2" H 4200 4600 50  0000 C CNN
 F 1 "green" H 4350 4550 50  0000 C CNN
 F 2 "LEDs:LED_0805_HandSoldering" H 4200 4500 50  0001 C CNN
@@
 $EndComp
 $Comp
-L device:LED D2
+L device:LED D1
 U 1 1 5A0E5A3A
 P 4950 4600
-F 0 "D2" H 4950 4700 50  0000 C CNN
+F 0 "D1" H 4950 4700 50  0000 C CNN
 F 1 "red" H 5100 4650 50  0000 C CNN
 F 2 "LEDs:LED_0805_HandSoldering" H 4950 4600 50  0001 C CNN

Commit message: Fixed symbol library references.
Parts:
- C1, C2, C6, C7: symbol device:C -> Device:C
- C3, C4, C5: symbol device:CP -> Device:CP
- D1, D2: symbol device:LED -> Device:LED
- J1: symbol conn:Conn_02x03_Odd_Even -> Connector_Generic:Conn_02x03_Odd_Even
- J2: symbol conn:Conn_01x05 -> Connector_Generic:Conn_01x05
- J3: symbol conn:Conn_01x03 -> Connector_Generic:Conn_01x03
- J4: symbol conn:DIN-6 -> Connector:DIN-6
- J5, J6: symbol hackup:C64-CassettePort -> hackup-commodore:C64-CassettePort
- J7: symbol conn:Conn_01x02 -> Connector_Generic:Conn_01x02
- J8: symbol conn:Conn_01x10 -> Connector_Generic:Conn_01x10
- R1, R10, R11, R12, R13, R14, R15, R16, R2, R3, R4, R5, R6, R7, R8, R9: symbol device:R -> Device:R
- U1: symbol atmel:ATMEGA644-20AU -> SD2IECplug:ATMEGA644-20AU-atmel
- U2: symbol regul:LM1117-3.3 -> Regulator_Linear:LM1117-3.3
- Y1: symbol device:Crystal -> Device:Crystal
Changed lines of the file:
@@
 EESchema Schematic File Version 4
 LIBS:SD2IECplug-cache
-EELAYER 26 0
+EELAYER 30 0
 EELAYER END
 $Descr A4 11693 8268
@@
 Sheet 1 1
 Title "SD2IEC Pluggable"
-Date "2018-10-14"
+Date "2019-12-18"
 Rev "2.1"
 Comp "www.hackup.net"
@@
 $EndDescr
 $Comp
-L atmel:ATMEGA644-20AU U1
+L SD2IECplug:ATMEGA644-20AU-atmel U1
 U 1 1 5A0DA765
 P 2400 4400
@@
 $EndComp
 $Comp
-L regul:LM1117-3.3 U2
+L Regulator_Linear:LM1117-3.3 U2
 U 1 1 5A0DA894
 P 9850 2400
@@
 $EndComp
 $Comp
-L device:C C6
+L Device:C C6
 U 1 1 5A0DB3FB
 P 10450 2550
@@
 $EndComp
 $Comp
-L conn:DIN-6 J4
+L Connector:DIN-6 J4
 U 1 1 5A0DB981
 P 10200 1200
@@
 IEC_ATN
 $Comp
-L device:Crystal Y1
+L Device:Crystal Y1
 U 1 1 5A0DC8F8
 P 1300 3300
@@
 $EndComp
 $Comp
-L device:C C1
+L Device:C C1
 U 1 1 5A0DCA05
 P 1000 3100
@@
 $EndComp
 $Comp
-L device:C C2
+L Device:C C2
 U 1 1 5A0DCA58
 P 1000 3500
@@
 $EndComp
 $Comp
-L device:R R12
+L Device:R R12
 U 1 1 5A0DEFAB
 P 6800 2150
@@
 $EndComp
 $Comp
-L device:R R14
+L Device:R R14
 U 1 1 5A0DF086
 P 7050 2150
@@
 $EndComp
 $Comp
-L device:R R13
+L Device:R R13
 U 1 1 5A0DF0C9
 P 7050 1600
@@
 $EndComp
 $Comp
-L device:R R9
+L Device:R R9
 U 1 1 5A0DF9C8
 P 5900 2150
@@
 $EndComp
 $Comp
-L device:R R11
+L Device:R R11
 U 1 1 5A0DF9CE
 P 6150 2150
@@
 $EndComp
 $Comp
-L device:R R10
+L Device:R R10
 U 1 1 5A0DF9D4
 P 6150 1600
@@
 $EndComp
 $Comp
-L device:R R6
+L Device:R R6
 U 1 1 5A0DFB40
 P 5000 2150
@@
 $EndComp
 $Comp
-L device:R R8
+L Device:R R8
 U 1 1 5A0DFB46
 P 5250 2150
@@
 $EndComp
 $Comp
-L device:R R7
+L Device:R R7
 U 1 1 5A0DFB4C
 P 5250 1600
@@
 $EndComp
 $Comp
-L device:R R2
+L Device:R R2
 U 1 1 5A0DFC58
 P 4100 2150
@@
 $EndComp
 $Comp
-L device:R R4
+L Device:R R4
 U 1 1 5A0DFC5E
 P 4350 2150
@@
 $EndComp
 $Comp
-L device:R R3
+L Device:R R3
 U 1 1 5A0DFC64
 P 4350 1600
@@
 SCK
 $Comp
-L conn:Conn_02x03_Odd_Even J1
+L Connector_Generic:Conn_02x03_Odd_Even J1
 U 1 1 5A0E128D
 P 1600 1300
@@
 $EndComp
 $Comp
-L device:CP C4
+L Device:CP C4
 U 1 1 5A0E450A
 P 9500 2550
@@
 $EndComp
 $Comp
-L device:CP C5
+L Device:CP C5
 U 1 1 5A0E45C6
 P 10200 2550
@@
 $EndComp
 $Comp
-L device:CP C3
+L Device:CP C3
 U 1 1 5A0E4A68
 P 8450 3750
@@
 $EndComp
 $Comp
-L device:R R1
+L Device:R R1
 U 1 1 5A0E56B2
 P 3800 4500
@@
 $EndComp
 $Comp
-L device:R R5
+L Device:R R5
 U 1 1 5A0E57F0
 P 4500 4600
@@
 $EndComp
 $Comp
-L device:LED D2
+L Device:LED D2
 U 1 1 5A0E5986
 P 4200 4500
@@
 $EndComp
 $Comp
-L device:LED D1
+L Device:LED D1
 U 1 1 5A0E5A3A
 P 4950 4600
@@
 $EndComp
 $Comp
-L device:R R15
+L Device:R R15
 U 1 1 5A0E7D80
 P 9400 3250
@@
 $EndComp
 $Comp
-L hackup:C64-CassettePort J5
+L hackup-commodore:C64-CassettePort J5
 U 1 1 5A140900
 P 2400 7700
@@
 Cas-Sense
 $Comp
-L hackup:C64-CassettePort J6
+L hackup-commodore:C64-CassettePort J6
 U 1 1 5A1416C4
 P 4300 7700
@@
 Wire Wire Line
 	9500 2700 9850 2700
-$Comp
-L conn:Conn_01x02 J7
-U 1 1 5B978294
-P 8850 2600
-F 0 "J7" H 8770 2275 50  0000 C CNN
-F 1 "Power" H 8770 2366 50  0000 C CNN
-F 2 "Pin_Headers:Pin_Header_Straight_1x02_Pitch2.54mm" H 8850 2600 50  0001 C CNN
-F 3 "~" H 8850 2600 50  0001 C CNN
-	1    8850 2600
-	-1   0    0    1
-$EndComp
 Wire Wire Line
 	9050 2500 9050 2400
@@
 Connection ~ 9500 2700
 Connection ~ 10450 2400
-$Comp
-L conn:Conn_01x10 J8
-U 1 1 5B9D412C
-P 7150 4650
-F 0 "J8" H 7250 5050 50  0000 L CNN
-F 1 "X3" H 7250 4150 50  0000 L CNN
-F 2 "Pin_Headers:Pin_Header_Straight_1x10_Pitch2.54mm" H 7150 4650 50  0001 C CNN
-F 3 "~" H 7150 4650 50  0001 C CNN
-	1    7150 4650
-	1    0    0    -1
-$EndComp
-$Comp
-L conn:Conn_01x05 J2
-U 1 1 5B9D4266
-P 5300 5150
-F 0 "J2" H 5450 4950 50  0000 C CNN
-F 1 "X6" H 5450 5350 50  0000 C CNN
-F 2 "Pin_Headers:Pin_Header_Straight_1x05_Pitch2.54mm" H 5300 5150 50  0001 C CNN
-F 3 "~" H 5300 5150 50  0001 C CNN
-	1    5300 5150
-	1    0    0    1
-$EndComp
 Wire Wire Line
 	6950 5050 6850 5050
@@
 $EndComp
 $Comp
-L conn:Conn_01x03 J3
-U 1 1 5B9BC1D8
-P 4450 3700
-F 0 "J3" H 4530 3742 50  0000 L CNN
-F 1 "Aux" H 4530 3651 50  0000 L CNN
-F 2 "Pin_Headers:Pin_Header_Straight_1x03_Pitch2.54mm" H 4450 3700 50  0001 C CNN
-F 3 "~" H 4450 3700 50  0001 C CNN
-	1    4450 3700
-	1    0    0    -1
-$EndComp
-$Comp
-L device:R R16
+L Device:R R16
 U 1 1 5B9BC306
 P 3750 3500
@@
 $EndComp
 $Comp
-L device:C C7
+L Device:C C7
 U 1 1 5BA17687
 P 1250 6300
@@
 Wire Wire Line
 	8750 1500 8750 1550
+$Comp
+L Connector_Generic:Conn_01x03 J3
+U 1 1 5B9BC1D8
+P 4450 3700
+F 0 "J3" H 4530 3742 50  0000 L CNN
+F 1 "Aux" H 4530 3651 50  0000 L CNN
+F 2 "Pin_Headers:Pin_Header_Straight_1x03_Pitch2.54mm" H 4450 3700 50  0001 C CNN
+F 3 "~" H 4450 3700 50  0001 C CNN
+	1    4450 3700
+	1    0    0    -1
+$EndComp
+$Comp
+L Connector_Generic:Conn_01x02 J7
+U 1 1 5B978294
+P 8850 2600
+F 0 "J7" H 8770 2275 50  0000 C CNN
+F 1 "Power" H 8770 2366 50  0000 C CNN
+F 2 "Pin_Headers:Pin_Header_Straight_1x02_Pitch2.54mm" H 8850 2600 50  0001 C CNN
+F 3 "~" H 8850 2600 50  0001 C CNN
+	1    8850 2600
+	-1   0    0    1
+$EndComp
+$Comp
+L Connector_Generic:Conn_01x10 J8
+U 1 1 5B9D412C
+P 7150 4650
+F 0 "J8" H 7250 5050 50  0000 L CNN
+F 1 "X3" H 7250 4150 50  0000 L CNN
+F 2 "Pin_Headers:Pin_Header_Straight_1x10_Pitch2.54mm" H 7150 4650 50  0001 C CNN
+F 3 "~" H 7150 4650 50  0001 C CNN
+	1    7150 4650
+	1    0    0    -1
+$EndComp
+$Comp
+L Connector_Generic:Conn_01x05 J2
+U 1 1 5B9D4266
+P 5300 5150
+F 0 "J2" H 5450 4950 50  0000 C CNN
+F 1 "X6" H 5450 5350 50  0000 C CNN
+F 2 "Pin_Headers:Pin_Header_Straight_1x05_Pitch2.54mm" H 5300 5150 50  0001 C CNN
+F 3 "~" H 5300 5150 50  0001 C CNN
+	1    5300 5150
+	1    0    0    1
+$EndComp
 $EndSCHEMATC

Commit message: Placement of C3 got messed up between v0.9 and v2.0, fixes #1.
Connections:
- net GND: now also C3.2, XS1.8 (DAT1)
Changed lines of the file:
@@
 EESchema Schematic File Version 4
-LIBS:SD2IECplug-cache
 EELAYER 30 0
 EELAYER END
@@
 Sheet 1 1
 Title "SD2IEC Pluggable"
-Date "2019-12-18"
-Rev "2.1"
+Date "2021-01-09"
+Rev "2.2"
 Comp "www.hackup.net"
 Comment1 ""
@@
 	9400 3400 9400 3475
 Wire Wire Line
-	9400 4775 9400 4800
-Wire Wire Line
 	3400 5600 8700 5600
 Wire Wire Line
 	3400 4000 8875 4000
 Wire Wire Line
-	8450 3900 8450 4300
+	8450 3900 8450 4150
 Wire Wire Line
 	8450 4300 8875 4300
@@
 Wire Wire Line
 	8700 4600 8700 5600
-Wire Wire Line
-	8875 4150 8575 4150
-Wire Wire Line
-	8575 4150 8575 4800
-Wire Wire Line
-	8575 4800 9400 4800
-Connection ~ 9400 4800
-Wire Wire Line
-	9400 4800 9400 4850
 $Comp
 L power:GND #PWR0103
@@
 	1    0    0    1
 $EndComp
+Wire Wire Line
+	9400 4775 9400 4800
+Wire Wire Line
+	9400 4800 8450 4800
+Wire Wire Line
+	8450 4800 8450 4300
+Connection ~ 9400 4800
+Wire Wire Line
+	9400 4800 9400 4850
+Connection ~ 8450 4300
+Wire Wire Line
+	8875 4150 8450 4150
+Connection ~ 8450 4150
+Wire Wire Line
+	8450 4150 8450 4300
 $EndSCHEMATC
